File: ts17-tropic01-mini.kicad_sch (KiCad schematic)
At the start: 9 parts, among them IC1 TROPIC01_chip, J1 Edge conn 4x 2.54, J2 Edge conn 4x 2.54

Commit message: Add manufacturing output files (gerber data and BOM)
Other:
- title: (none) -> TROPIC01 integration board "mini"
Changed lines of the file:
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@@
 	(generator_version "9.0")
 	(paper "A4")
+	(title_block
+		(title "TROPIC01 integration board \"mini\"")
+		(date "2025-11-07")
+		(rev "TS1701")
+	)
 	(text "5"
 		(exclude_from_sim no)
